File: kicad_prototipe1/prototipe1.kicad_pcb (KiCad board)
At the start: 2 copper layers, 68.6 x 53.3 mm, 12 parts, among them P1 Power, P2 Analog, P3 Digital, P4 Digital, P5 CONN_01X01, P6 CONN_01X01, P7 CONN_01X01, P8 CONN_01X01

Commit message: update kicad prototipe1
Parts:
- moved DCMotor1 12.7 mm to (169.4, 98.4), turned to 180 degrees
- moved GY-87 10.5 mm to (135.1, 113.7), turned to 180 degrees
- moved DCMotor2 4.58 mm to (158.0, 98.4)
Connections:
- L298N_INPUT1 pad 1: /9(**) -> /5(**)
- L298N_INPUT1 pad 2: /4 -> /6(**)
- L298N_INPUT1 pad 3: /5(**) -> /7
- L298N_INPUT1 pad 4: /6(**) -> /8
- L298N_INPUT1 pad 5: /7 -> /9(**)
Routing:
- net GND: track 154.6 -> 94.5 mm
- net +5V: track 50.6 -> 77.1 mm
- net /4: track 21.5 -> 0.00 mm
- net /3(**): track 43.4 -> 25.2 mm
- net /7: track 30.6 -> 15.7 mm
- net /8: track 0.00 -> 14.3 mm
- net +3V3: track 14.3 -> 27.6 mm
- net /A4(SDA): track 42.1 -> 29.1 mm
- net /A5(SCL): track 42.1 -> 32.7 mm
- net /6(**): track 21.5 -> 15.7 mm
- net /5(**): track 21.5 -> 15.7 mm
- net /2: track 10.8 -> 15.6 mm
- net /0(Rx): track 22.4 -> 17.7 mm
- net /9(**): track 10.3 -> 14.3 mm
- net /1(Tx): track 15.9 -> 19.2 mm
- removed copper zone on F.Cu, net +5V
Other:
- board size 68.6 x 53.3 mm -> 68.6 x 55.9 mm
