File: kicad_prototipe1/prototipe1.kicad_sch (KiCad schematic)
At the start: 12 parts, among them P1 Power, P2 Analog, P3 Digital, P4 Digital, P5 CONN_01X01, P6 CONN_01X01, P7 CONN_01X01, P8 CONN_01X01

Commit message: update kicad prototipe1
Connections:
- net 4: no longer L298N_INPUT1.2 (Pin_2)
- net 5(**): now also L298N_INPUT1.1 (Pin_1); no longer L298N_INPUT1.3 (Pin_3)
- net 6(**): now also L298N_INPUT1.2 (Pin_2); no longer L298N_INPUT1.4 (Pin_4)
- net 7: now also L298N_INPUT1.3 (Pin_3); no longer L298N_INPUT1.5 (Pin_5)
- net 8: now also L298N_INPUT1.4 (Pin_4)
- net 9(**): now also L298N_INPUT1.5 (Pin_5); no longer L298N_INPUT1.1 (Pin_1)
Changed lines of the file:
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@@
+    (stroke (width 0) (type default) (color 0 0 0 0))
+  )
+  (wire (pts (xy 119.38 43.18) (xy 125.73 43.18))
     (stroke (width 0) (type default) (color 0 0 0 0))
   )
@@
     (stroke (width 0) (type solid) (color 0 0 0 0))
   )
+  (wire (pts (xy 119.38 33.02) (xy 125.73 33.02))
+    (stroke (width 0) (type default) (color 0 0 0 0))
+  )
   (wire (pts (xy 259.08 43.18) (xy 267.97 43.18))
     (stroke (width 0) (type solid) (color 0 0 0 0))
@@
     (stroke (width 0) (type solid) (color 0 0 0 0))
   )
+  (wire (pts (xy 119.38 38.1) (xy 125.73 38.1))
+    (stroke (width 0) (type default) (color 0 0 0 0))
+  )
   (wire (pts (xy 119.38 63.5) (xy 137.16 63.5))
     (stroke (width 0) (type default) (color 0 0 0 0))
@@
     (stroke (width 0) (type solid) (color 0 0 0 0))
   )
-  (wire (pts (xy 119.38 33.02) (xy 125.73 33.02))
-    (stroke (width 0) (type default) (color 0 0 0 0))
-  )
   (wire (pts (xy 156.21 27.94) (xy 167.64 27.94))
     (stroke (width 0) (type default) (color 0 0 0 0))
@@
     (stroke (width 0) (type default) (color 0 0 0 0))
   )
+  (wire (pts (xy 236.22 55.88) (xy 236.22 80.01))
+    (stroke (width 0) (type solid) (color 0 0 0 0))
+  )
+  (wire (pts (xy 227.33 58.42) (xy 227.33 36.83))
+    (stroke (width 0) (type solid) (color 0 0 0 0))
+  )
+  (wire (pts (xy 119.38 35.56) (xy 125.73 35.56))
+    (stroke (width 0) (type default) (color 0 0 0 0))
+  )
+  (polyline (pts (xy 215.9 87.63) (xy 284.48 87.63))
+    (stroke (width 0) (type dash) (color 0 0 0 0))
+  )
+  (wire (pts (xy 259.08 68.58) (xy 267.97 68.58))
+    (stroke (width 0) (type solid) (color 0 0 0 0))
+  )
+  (wire (pts (xy 238.76 76.2) (xy 226.06 76.2))
+    (stroke (width 0) (type solid) (color 0 0 0 0))
+  )
+  (wire (pts (xy 259.08 73.66) (xy 267.97 73.66))
+    (stroke (width 0) (type solid) (color 0 0 0 0))
+  )
+  (polyline (pts (xy 271.78 25.4) (xy 271.78 12.7))
+    (stroke (width 0) (type dash) (color 0 0 0 0))
+  )
+  (wire (pts (xy 259.08 60.96) (xy 267.97 60.96))
+    (stroke (width 0) (type solid) (color 0 0 0 0))
+  )
+  (wire (pts (xy 119.38 40.64) (xy 125.73 40.64))
+    (stroke (width 0) (type default) (color 0 0 0 0))
+  )
+  (wire (pts (xy 229.87 50.8) (xy 229.87 34.29))
+    (stroke (width 0) (type solid) (color 0 0 0 0))
+  )
+  (wire (pts (xy 119.38 66.04) (xy 137.16 66.04))
+    (stroke (width 0) (type default) (color 0 0 0 0))
+  )
+  (wire (pts (xy 259.08 33.02) (xy 267.97 33.02))
+    (stroke (width 0) (type solid) (color 0 0 0 0))
+  )
+  (wire (pts (xy 259.08 66.04) (xy 267.97 66.04))
+    (stroke (width 0) (type solid) (color 0 0 0 0))
+  )
+  (wire (pts (xy 259.08 35.56) (xy 267.97 35.56))
+    (stroke (width 0) (type solid) (color 0 0 0 0))
+  )
+  (polyline (pts (xy 215.9 12.7) (xy 215.9 87.63))
+    (stroke (width 0) (type dash) (color 0 0 0 0))
+  )
+  (wire (pts (xy 232.41 48.26) (xy 232.41 36.83))
+    (stroke (width 0) (type solid) (color 0 0 0 0))
+  )
+  (wire (pts (xy 237.49 36.83) (xy 237.49 43.18))
+    (stroke (width 0) (type solid) (color 0 0 0 0))
+  )
+  (wire (pts (xy 259.08 76.2) (xy 267.97 76.2))
+    (stroke (width 0) (type solid) (color 0 0 0 0))
+  )
+  (wire (pts (xy 259.08 48.26) (xy 267.97 48.26))
+    (stroke (width 0) (type solid) (color 0 0 0 0))
+  )
+  (wire (pts (xy 238.76 68.58) (xy 226.06 68.58))
+    (stroke (width 0) (type solid) (color 0 0 0 0))
+  )
   (wire (pts (xy 119.38 45.72) (xy 125.73 45.72))
     (stroke (width 0) (type default) (color 0 0 0 0))
-  )
-  (wire (pts (xy 236.22 55.88) (xy 236.22 80.01))
-    (stroke (width 0) (type solid) (color 0 0 0 0))
-  )
-  (wire (pts (xy 227.33 58.42) (xy 227.33 36.83))
-    (stroke (width 0) (type solid) (color 0 0 0 0))
-  )
-  (wire (pts (xy 119.38 38.1) (xy 125.73 38.1))
-    (stroke (width 0) (type default) (color 0 0 0 0))
-  )
-  (polyline (pts (xy 215.9 87.63) (xy 284.48 87.63))
-    (stroke (width 0) (type dash) (color 0 0 0 0))
-  )
-  (wire (pts (xy 119.38 43.18) (xy 125.73 43.18))
-    (stroke (width 0) (type default) (color 0 0 0 0))
-  )
-  (wire (pts (xy 259.08 68.58) (xy 267.97 68.58))
-    (stroke (width 0) (type solid) (color 0 0 0 0))
-  )
-  (wire (pts (xy 238.76 76.2) (xy 226.06 76.2))
-    (stroke (width 0) (type solid) (color 0 0 0 0))
-  )
-  (wire (pts (xy 259.08 73.66) (xy 267.97 73.66))
-    (stroke (width 0) (type solid) (color 0 0 0 0))
-  )
-  (polyline (pts (xy 271.78 25.4) (xy 271.78 12.7))
-    (stroke (width 0) (type dash) (color 0 0 0 0))
-  )
-  (wire (pts (xy 259.08 60.96) (xy 267.97 60.96))
-    (stroke (width 0) (type solid) (color 0 0 0 0))
-  )
-  (wire (pts (xy 229.87 50.8) (xy 229.87 34.29))
-    (stroke (width 0) (type solid) (color 0 0 0 0))
-  )
-  (wire (pts (xy 119.38 66.04) (xy 137.16 66.04))
-    (stroke (width 0) (type default) (color 0 0 0 0))
-  )
-  (wire (pts (xy 259.08 33.02) (xy 267.97 33.02))
-    (stroke (width 0) (type solid) (color 0 0 0 0))
-  )
-  (wire (pts (xy 259.08 66.04) (xy 267.97 66.04))
-    (stroke (width 0) (type solid) (color 0 0 0 0))
-  )
-  (wire (pts (xy 259.08 35.56) (xy 267.97 35.56))
-    (stroke (width 0) (type solid) (color 0 0 0 0))
-  )
-  (wire (pts (xy 119.38 40.64) (xy 125.73 40.64))
-    (stroke (width 0) (type default) (color 0 0 0 0))
-  )
-  (polyline (pts (xy 215.9 12.7) (xy 215.9 87.63))
-    (stroke (width 0) (type dash) (color 0 0 0 0))
-  )
-  (wire (pts (xy 232.41 48.26) (xy 232.41 36.83))
-    (stroke (width 0) (type solid) (color 0 0 0 0))
-  )
-  (wire (pts (xy 237.49 36.83) (xy 237.49 43.18))
-    (stroke (width 0) (type solid) (color 0 0 0 0))
-  )
-  (wire (pts (xy 259.08 76.2) (xy 267.97 76.2))
-    (stroke (width 0) (type solid) (color 0 0 0 0))
-  )
-  (wire (pts (xy 259.08 48.26) (xy 267.97 48.26))
-    (stroke (width 0) (type solid) (color 0 0 0 0))
-  )
-  (wire (pts (xy 119.38 35.56) (xy 125.73 35.56))
-    (stroke (width 0) (type default) (color 0 0 0 0))
-  )
-  (wire (pts (xy 238.76 68.58) (xy 226.06 68.58))
-    (stroke (width 0) (type solid) (color 0 0 0 0))
   )
   (polyline (pts (xy 216.535 20.955) (xy 252.095 20.955))
@@
     (effects (font (size 1.524 1.524)) (justify left bottom))
   )
+  (label "8" (at 125.73 40.64 0)
+    (effects (font (size 1.524 1.524)) (justify left bottom))
+  )
   (label "A5(SCL)" (at 226.06 76.2 0)
     (effects (font (size 1.524 1.524)) (justify left bottom))
@@
     (effects (font (size 1.524 1.524)) (justify left bottom))
   )
-  (label "4" (at 125.73 35.56 0)
-    (effects (font (size 1.524 1.524)) (justify left bottom))
-  )
   (label "3(**)" (at 267.97 68.58 0)
     (effects (font (size 1.524 1.524)) (justify left bottom))
@@
     (effects (font (size 1.27 1.27)) (justify left bottom))
   )
-  (label "7" (at 125.73 43.18 0)
+  (label "7" (at 125.73 38.1 0)
     (effects (font (size 1.524 1.524)) (justify left bottom))
   )
@@
     (effects (font (size 1.524 1.524)) (justify left bottom))
   )
-  (label "5(**)" (at 125.73 38.1 0)
-    (effects (font (size 1.524 1.524)) (justify left bottom))
-  )
-  (label "9(**)" (at 125.73 33.02 0)
+  (label "5(**)" (at 125.73 33.02 0)
+    (effects (font (size 1.524 1.524)) (justify left bottom))
+  )
+  (label "9(**)" (at 125.73 43.18 0)
     (effects (font (size 1.524 1.524)) (justify left bottom))
   )
@@
     (effects (font (size 1.524 1.524)) (justify left bottom))
   )
-  (label "6(**)" (at 125.73 40.64 0)
-    (effects (font (size 1.524 1.524)) (justify left bottom))
-  )
+  (label "6(**)" (at 125.73 35.56 0)
+    (effects (font (size 1.524 1.524)) (justify left bottom))
+  )
